File: hardware/IgnisV2/IgnisV2.kicad_sch (KiCad schematic)
At the start: 0 parts

Commit message: 🎨 Complete logo cleanup and rebranding with new typography
- Changed official logo font from Museo Rounded to "Dongle" Bold
- Reorganized logo assets with consistent naming convention
- Added Makefile for automated PNG export in multiple variants and sizes
- Updated KiCAD worksheets for both IgnisV1 and IgnisV2 PCBs with new branding
- Removed obsolete logo files and consolidated SVG sources
- Exported updated schematic PDFs with refreshed corporate identity
Other:
- title: (none) -> Ignis
