File: hardware/IgnisV2/power_stage.kicad_sch (KiCad schematic)
At the start: 55 parts, among them J1 COIL_A, J2 COIL_B, J3 530480210, U1 BQ51013BRHLT, U2 BQ24073RGTR, U3 FP6277XR-G1

Commit message: 🏭 Finalize IgnisV2 PCB design and prepare for JLCPCB production
- Polished hierarchical schematics with clean signal routing
- Completed full PCB layout with optimized component placement
- Refined component selection for optimal JLCPCB compatibility
- Generated production files (Gerbers, drill, BOM, pick&place) for fabrication
- Exported 3D model snapshot for documentation and review
- Added 74LVC1G17 datasheet for package selection reference
- Selected TSSOP-5 package over SOT1202 for PCBA compatibility
- Configured for advanced PCBA service due to WS2812B backing requirements
- Updated design rules and gitignore for production workflow
Parts:
- removed TP10: FB, TestPoint:TestPoint_Pad_D1.0mm, symbol Connector:TestPoint_Flag
- J1, J2: footprint Connector_Wire:SolderWire-0.25sqmm_1x01_D0.65mm_OD1.7mm -> TestPoint:TestPoint_THTPad_D1.5mm_Drill0.7mm
- JP1: value VGNDC -> VBATS
- JP2: value VBATC -> VGNDS
Connections:
- net ~{STBY} is gone; now on net ~{PGOOD}: R9.2
- net GND: now also U2.18 (EXP), U2.19 (EXP), U2.20 (EXP), U2.21 (EXP), U2.22 (EXP)
- net AC2: now reaches C11.1, C3.1, C4.1, C7.1, C9.1, J2.1 (Pin_1), TP2.1, U1.19 (AC2)
- net AC1: now reaches C1.2, C10.1, C2.2, C3.2, C4.2, C5.2, C6.1, C8.1, U1.2 (AC1)
- net VBAT: now reaches C18.1, JP1.2 (C), TP5.1, U2.2 (BAT), U2.3 (BAT)
- net COILA: now reaches C1.1, C2.1, C5.1, J1.1 (Pin_1), TP1.1
- net at JP1.1 (A), JP2.3 (B): now also J3.2 (VBAT); no longer J3.1
- net at JP1.3 (B), JP2.1 (A): now also J3.1 (GND); no longer J3.2

Commit message: 🎨 Complete logo cleanup and rebranding with new typography
- Changed official logo font from Museo Rounded to "Dongle" Bold
- Reorganized logo assets with consistent naming convention
- Added Makefile for automated PNG export in multiple variants and sizes
- Updated KiCAD worksheets for both IgnisV1 and IgnisV2 PCBs with new branding
- Removed obsolete logo files and consolidated SVG sources
- Exported updated schematic PDFs with refreshed corporate identity
Other:
- title: (none) -> Ignis
Changed lines of the file:
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@@
 	(generator_version "9.0")
 	(paper "A4")
+	(title_block
+		(title "Ignis")
+		(date "2025-08-26")
+		(rev "v2.2")
+	)
 	(text_box "Inductive Charger"
 		(exclude_from_sim no)
